Commit message: bug fix

File: src/gemstone_bringup/urdf/gemstone_ugv.urdf.xacro (robot description, xacro)
@@ -111,5 +111,5 @@
     <parent link="base_link"/>
     <child link="lidar_link"/>
-    <origin xyz="0 0 ${chassis_height/2 + 0.05}" rpy="0 0 0"/>
+    <origin xyz="0 0 ${chassis_height/2 + 0.05}" rpy="0 0 2.068"/>
   </joint>
   <link name="camera_link"/>
