Commit message: feat: restructure UGV into a 3-tier chassis in the sim model
The Gazebo model now matches the real build layout:

- BOTTOM tier (base_link): chassis plate, encoder drive wheels on both
  sides, caster, 3S LiPo battery in the center
- MIDDLE tier (mid_plate): gemstone O1 board + motor driver
- TOP tier (top_plate): A1M8 lidar on top, camera on the front edge below
  the lidar plane

Fixes:
- Sensor links (lidar/camera/imu) are attached directly to base_link via
  their fixed-joint origins. With a multi-level fixed-joint chain, the
  URDF->SDF conversion kept the sensor at the root link origin (0,0,0),
  so the lidar emitted from the chassis instead of the top tier.
- Camera moved below the lidar scan plane so the front rays are not
  blocked.

Verified in sim: /scan now returns office geometry (1.9-3.5 m ranges,
no sub-0.5 m self-occlusion), exploration picks targets at 2-3.5 m, and
sensors sit at z = 0.155 (lidar), 0.12 (camera), 0.105 (imu).

Co-authored-by: alitalhq <alitqlhq@gmail.com>

File: src/gemstone_sim/urdf/gemstone_ugv_gazebo.xacro (robot description, xacro)
@@ -2,24 +2,33 @@
 <robot name="gemstone_ugv_gazebo" xmlns:xacro="http://www.ros.org/wiki/xacro">
   <!--
-    Gemstone UGV'nin Gazebo Classic simülasyonuna uygun hali.
+    Gemstone UGV'nin Gazebo Classic simülasyonuna uygun 3 katli hali.
     Gerçek robot URDF'i (gemstone_bringup/urdf/gemstone_ugv.urdf.xacro) ile
     aynı kinematik yapı (2 tahrik tekeri + 1 ön misket teker) kullanılır.
+    3 katli mekanik yapi (asagidan yukari):
+      - ALT KAT   : şasi tablasi + iki yanda encoder'li tahrik tekerleri +
+                    ortada 3S LiPo pil
+      - ORTA KAT  : gemstone (O1) karti + motor surucu (platformun uzerinde)
+      - UST KAT   : A1M8 lidar (platform uzerinde, en tepede)
+    ONEMLI: Her katmanın yerlesimi JOINT origin'inde tasinir; boylece her
+    linkin FRAME'i kendi katinda durur. Sensörler (<gazebo reference> ile
+    eklenen ray/imu/camera) linkin FRAME orijininden yayilir - eger joint
+    origin'i tasimazsaniz sensörler base_link orijininde (en altta) kalir.
     Farklar:
-      - Ölçüler fizik/denge için hafif düzeltildi (orijinal xacro'daki
-        değerler zaten "yer tutucu" idi). Tekerler şasinin altından taşar ve
-        robot yerde dengede durur (3 nokta: 2 teker + 1 misket).
+      - Ölçüler fizik/denge için hafif düzeltildi. Tekerler şasinin altından
+        taşar ve robot yerde dengede durur (3 nokta: 2 teker + 1 misket).
       - gazebo_ros plugin'leri eklendi:
           * diff_drive        -> /cmd_vel dinler, /odom + odom->base_link TF yayinlar
           * gpu/cpu ray lidar -> /scan (360 ornek, 3.5 m, RPLidar A1M8 benzeri)
-          * imu_sensor        -> /imu/data
-          * camera            -> /camera/image_raw
+          * imu_sensor        -> /imu/data (gemstone kartinin uzerinde)
+          * camera            -> /camera/image_raw (lidar duzleminin altinda)
           * joint_state       -> /joint_states (robot_state_publisher icin)
       - Tekerlekler yere tutunmasi icin yuksek surtunme (mu=100000) tanimli.
   -->
   <!-- ======================= Yer tutucu olculer (sim) ======================= -->
+  <!-- Alt kapi (base_link) tablasi -->
   <xacro:property name="chassis_length" value="0.30"/>
   <xacro:property name="chassis_width" value="0.20"/>
-  <xacro:property name="chassis_height" value="0.06"/>
-  <xacro:property name="chassis_mass" value="2.0"/>
+  <xacro:property name="chassis_thickness" value="0.03"/>
+  <xacro:property name="chassis_mass" value="1.0"/>
   <xacro:property name="wheel_radius" value="0.065"/>
   <xacro:property name="wheel_width" value="0.04"/>
@@ -33,4 +42,43 @@
   <xacro:property name="caster_x_offset" value="0.12"/>
   <xacro:property name="caster_z_offset" value="-0.055"/>
+  <!-- 3S LiPo pil (alt katin ortasinda) -->
+  <xacro:property name="battery_length" value="0.14"/>
+  <xacro:property name="battery_width" value="0.09"/>
+  <xacro:property name="battery_height" value="0.025"/>
+  <xacro:property name="battery_z" value="${chassis_thickness/2 + battery_height/2}"/>
+  <xacro:property name="battery_mass" value="0.25"/>
+  <!-- Orta kapi tablasi (gemstone + motor surucu) -->
+  <xacro:property name="mid_plate_length" value="0.28"/>
+  <xacro:property name="mid_plate_width" value="0.18"/>
+  <xacro:property name="mid_plate_thickness" value="0.03"/>
+  <xacro:property name="mid_plate_z" value="${chassis_thickness/2 + 0.04 + mid_plate_thickness/2}"/>
+  <xacro:property name="mid_plate_mass" value="0.8"/>
+  <!-- Gemstone O1 karti ve motor surucu (orta katin uzerinde) -->
+  <xacro:property name="board_length" value="0.08"/>
+  <xacro:property name="board_width" value="0.06"/>
+  <xacro:property name="board_thickness" value="0.015"/>
+  <xacro:property name="board_z" value="${mid_plate_z + mid_plate_thickness/2 + board_thickness/2}"/>
+  <xacro:property name="board_mass" value="0.05"/>
+  <xacro:property name="driver_length" value="0.05"/>
+  <xacro:property name="driver_width" value="0.04"/>
+  <xacro:property name="driver_thickness" value="0.015"/>
+  <xacro:property name="driver_x" value="0.055"/>
+  <xacro:property name="driver_z" value="${board_z}"/>
+  <xacro:property name="driver_mass" value="0.05"/>
+  <!-- Ust kapi tablasi (A1M8 lidar) -->
+  <xacro:property name="top_plate_length" value="0.22"/>
+  <xacro:property name="top_plate_width" value="0.16"/>
+  <xacro:property name="top_plate_thickness" value="0.02"/>
+  <xacro:property name="top_plate_z" value="${board_z + board_thickness/2 + 0.02 + top_plate_thickness/2}"/>
+  <xacro:property name="top_plate_mass" value="0.6"/>
+  <!-- A1M8 lidar (ust katin uzerinde, en tepede) -->
+  <xacro:property name="lidar_radius" value="0.026"/>
+  <xacro:property name="lidar_height" value="0.03"/>
+  <xacro:property name="lidar_z" value="${top_plate_z + top_plate_thickness/2 + lidar_height/2}"/>
+  <xacro:property name="lidar_mass" value="0.10"/>
+  <!-- Kamera: ust katin on kenarinda, lidar duzleminin ALTINDA kalsin ki
+       lidar ışınlarını engellemesin (lidar duzlemi z=lidar_z civarinda) -->
+  <xacro:property name="camera_x" value="${top_plate_length/2 + 0.015}"/>
+  <xacro:property name="camera_z" value="${top_plate_z - 0.01}"/>
   <material name="gemstone_gray">
     <color rgba="0.45 0.48 0.5 1.0"/>
@@ -42,9 +90,18 @@
     <color rgba="0.9 0.9 0.9 1.0"/>
   </material>
-  <!-- ================================ Şasi ================================ -->
+  <material name="battery_red">
+    <color rgba="0.55 0.08 0.08 1.0"/>
+  </material>
+  <material name="pcb_green">
+    <color rgba="0.1 0.55 0.2 1.0"/>
+  </material>
+  <material name="driver_blue">
+    <color rgba="0.1 0.3 0.7 1.0"/>
+  </material>
+  <!-- ================= ALT KAT: Şasi tablasi (base_link) ================= -->
   <link name="base_link">
     <visual>
       <geometry>
-        <box size="${chassis_length} ${chassis_width} ${chassis_height}"/>
+        <box size="${chassis_length} ${chassis_width} ${chassis_thickness}"/>
       </geometry>
       <material name="gemstone_gray"/>
@@ -52,13 +109,36 @@
     <collision>
       <geometry>
-        <box size="${chassis_length} ${chassis_width} ${chassis_height}"/>
+        <box size="${chassis_length} ${chassis_width} ${chassis_thickness}"/>
       </geometry>
     </collision>
     <inertial>
       <mass value="${chassis_mass}"/>
-      <inertia ixx="0.01" ixy="0.0" ixz="0.0" iyy="0.02" iyz="0.0" izz="0.02"/>
-    </inertial>
-  </link>
-  <!-- ============================ Tahrik tekerleri ============================ -->
+      <inertia ixx="0.0034" ixy="0.0" ixz="0.0" iyy="0.0076" iyz="0.0" izz="0.0108"/>
+    </inertial>
+  </link>
+  <!-- 3S LiPo pil: alt katin ortasinda -->
+  <link name="battery_link">
+    <visual>
+      <geometry>
+        <box size="${battery_length} ${battery_width} ${battery_height}"/>
+      </geometry>
+      <material name="battery_red"/>
+    </visual>
+    <collision>
+      <geometry>
+        <box size="${battery_length} ${battery_width} ${battery_height}"/>
+      </geometry>
+    </collision>
+    <inertial>
+      <mass value="${battery_mass}"/>
+      <inertia ixx="0.00018" ixy="0.0" ixz="0.0" iyy="0.00042" iyz="0.0" izz="0.00058"/>
+    </inertial>
+  </link>
+  <joint name="battery_joint" type="fixed">
+    <parent link="base_link"/>
+    <child link="battery_link"/>
+    <origin xyz="0 0 ${battery_z}" rpy="0 0 0"/>
+  </joint>
+  <!-- ===================== ALT KAT: Tahrik tekerleri ===================== -->
   <xacro:macro name="drive_wheel" params="prefix y_reflect">
     <link name="${prefix}_wheel_link">
@@ -99,5 +179,5 @@
   <xacro:drive_wheel prefix="left" y_reflect="1"/>
   <xacro:drive_wheel prefix="right" y_reflect="-1"/>
-  <!-- ============================ Misket (caster) teker ============================ -->
+  <!-- ===================== ALT KAT: Misket (caster) teker ===================== -->
   <link name="caster_wheel_link">
     <visual>
@@ -122,9 +202,158 @@
     <origin xyz="${caster_x_offset} 0 ${caster_z_offset}" rpy="0 0 0"/>
   </joint>
-  <!-- ============================ Sensör çerçeveleri ============================ -->
+  <!-- ===================== ORTA KAT: platform tablasi ===================== -->
+  <link name="mid_plate_link">
+    <visual>
+      <geometry>
+        <box size="${mid_plate_length} ${mid_plate_width} ${mid_plate_thickness}"/>
+      </geometry>
+      <material name="gemstone_gray"/>
+    </visual>
+    <collision>
+      <geometry>
+        <box size="${mid_plate_length} ${mid_plate_width} ${mid_plate_thickness}"/>
+      </geometry>
+    </collision>
+    <inertial>
+      <mass value="${mid_plate_mass}"/>
+      <inertia ixx="0.00222" ixy="0.0" ixz="0.0" iyy="0.00529" iyz="0.0" izz="0.00739"/>
+    </inertial>
+  </link>
+  <joint name="mid_plate_joint" type="fixed">
+    <parent link="base_link"/>
+    <child link="mid_plate_link"/>
+    <origin xyz="0 0 ${mid_plate_z}" rpy="0 0 0"/>
+  </joint>
+  <!-- Gemstone O1 karti: orta katin uzerinde -->
+  <link name="gemstone_link">
+    <visual>
+      <geometry>
+        <box size="${board_length} ${board_width} ${board_thickness}"/>
+      </geometry>
+      <material name="pcb_green"/>
+    </visual>
+    <collision>
+      <geometry>
+        <box size="${board_length} ${board_width} ${board_thickness}"/>
+      </geometry>
+    </collision>
+    <inertial>
+      <mass value="${board_mass}"/>
+      <inertia ixx="0.000016" ixy="0.0" ixz="0.0" iyy="0.000028" iyz="0.0" izz="0.000042"/>
+    </inertial>
+  </link>
+  <joint name="gemstone_joint" type="fixed">
+    <parent link="mid_plate_link"/>
+    <child link="gemstone_link"/>
+    <origin xyz="0 0 ${board_z}" rpy="0 0 0"/>
+  </joint>
+  <!-- Motor surucu: gemstone kartinin yaninda -->
+  <link name="motor_driver_link">
+    <visual>
+      <geometry>
+        <box size="${driver_length} ${driver_width} ${driver_thickness}"/>
+      </geometry>
+      <material name="driver_blue"/>
+    </visual>
+    <collision>
+      <geometry>
+        <box size="${driver_length} ${driver_width} ${driver_thickness}"/>
+      </geometry>
+    </collision>
+    <inertial>
+      <mass value="${driver_mass}"/>
+      <inertia ixx="0.000008" ixy="0.0" ixz="0.0" iyy="0.000012" iyz="0.0" izz="0.000018"/>
+    </inertial>
+  </link>
+  <joint name="motor_driver_joint" type="fixed">
+    <parent link="mid_plate_link"/>
+    <child link="motor_driver_link"/>
+    <origin xyz="${driver_x} 0 ${driver_z}" rpy="0 0 0"/>
+  </joint>
+  <!-- ===================== UST KAT: platform tablasi ===================== -->
+  <link name="top_plate_link">
+    <visual>
+      <geometry>
+        <box size="${top_plate_length} ${top_plate_width} ${top_plate_thickness}"/>
+      </geometry>
+      <material name="gemstone_gray"/>
+    </visual>
+    <collision>
+      <geometry>
+        <box size="${top_plate_length} ${top_plate_width} ${top_plate_thickness}"/>
+      </geometry>
+    </collision>
+    <inertial>
+      <mass value="${top_plate_mass}"/>
+      <inertia ixx="0.00130" ixy="0.0" ixz="0.0" iyy="0.00244" iyz="0.0" izz="0.00370"/>
+    </inertial>
+  </link>
+  <joint name="top_plate_joint" type="fixed">
+    <parent link="mid_plate_link"/>
+    <child link="top_plate_link"/>
+    <origin xyz="0 0 ${top_plate_z}" rpy="0 0 0"/>
+  </joint>
+  <!-- A1M8 lidar: ust katin uzerinde, en tepede -->
+  <link name="lidar_link">
+    <visual>
+      <geometry>
+        <cylinder radius="${lidar_radius}" length="${lidar_height}"/>
+      </geometry>
+      <material name="gemstone_black"/>
+    </visual>
+    <collision>
+      <geometry>
+        <cylinder radius="${lidar_radius}" length="${lidar_height}"/>
+      </geometry>
+    </collision>
+    <inertial>
+      <mass value="${lidar_mass}"/>
+      <inertia ixx="0.000025" ixy="0.0" ixz="0.0" iyy="0.000025" iyz="0.0" izz="0.000034"/>
+    </inertial>
+  </link>
+  <joint name="lidar_joint" type="fixed">
+    <parent link="base_link"/>
+    <child link="lidar_link"/>
+    <origin xyz="0 0 ${lidar_z}" rpy="0 0 0"/>
+  </joint>
+  <!-- ===================== Kamera (ust kat, onde) ===================== -->
+  <link name="camera_link">
+    <visual>
+      <geometry>
+        <box size="0.03 0.02 0.02"/>
+      </geometry>
+      <material name="gemstone_black"/>
+    </visual>
+    <collision>
+      <geometry>
+        <box size="0.03 0.02 0.02"/>
+      </geometry>
+    </collision>
+    <inertial>
+      <mass value="0.02"/>
+      <inertia ixx="0.0000013" ixy="0.0" ixz="0.0" iyy="0.0000013" iyz="0.0" izz="0.0000022"/>
+    </inertial>
+  </link>
+  <joint name="camera_joint" type="fixed">
+    <parent link="base_link"/>
+    <child link="camera_link"/>
+    <origin xyz="${camera_x} 0 ${camera_z}" rpy="0 0 0"/>
+  </joint>
+  <!-- ===================== IMU (gemstone karti uzerinde) ===================== -->
   <link name="imu_link">
+    <visual>
+      <geometry>
+        <box size="0.02 0.02 0.01"/>
+      </geometry>
+      <material name="gemstone_white"/>
+    </visual>
+    <collision>
+      <geometry>
+        <box size="0.02 0.02 0.01"/>
+      </geometry>
+    </collision>
     <inertial>
       <mass value="0.01"/>
-      <inertia ixx="0.00001" ixy="0.0" ixz="0.0" iyy="0.00001" iyz="0.0" izz="0.00001"/>
+      <inertia ixx="0.000001" ixy="0.0" ixz="0.0" iyy="0.000001" iyz="0.0" izz="0.000001"/>
     </inertial>
   </link>
@@ -132,27 +361,5 @@
     <parent link="base_link"/>
     <child link="imu_link"/>
-    <origin xyz="0 0 0" rpy="0 0 0"/>
-  </joint>
-  <link name="lidar_link">
-    <inertial>
-      <mass value="0.01"/>
-      <inertia ixx="0.00001" ixy="0.0" ixz="0.0" iyy="0.00001" iyz="0.0" izz="0.00001"/>
-    </inertial>
-  </link>
-  <joint name="lidar_joint" type="fixed">
-    <parent link="base_link"/>
-    <child link="lidar_link"/>
-    <origin xyz="0 0 ${chassis_height/2 + 0.05}" rpy="0 0 0"/>
-  </joint>
-  <link name="camera_link">
-    <inertial>
-      <mass value="0.01"/>
-      <inertia ixx="0.00001" ixy="0.0" ixz="0.0" iyy="0.00001" iyz="0.0" izz="0.00001"/>
-    </inertial>
-  </link>
-  <joint name="camera_joint" type="fixed">
-    <parent link="base_link"/>
-    <child link="camera_link"/>
-    <origin xyz="${chassis_length/2} 0 ${chassis_height/2}" rpy="0 0 0"/>
+    <origin xyz="0 0 ${board_z + board_thickness/2 + 0.005}" rpy="0 0 0"/>
   </joint>
   <!-- ============================ Sensörler ============================ -->

Commit message: fix: correct mid-plate children placement and add visual materials
The middle-tier children (gemstone, motor driver, top plate) used
absolute heights in their joint origins, but these joints are relative
to mid_plate_link. Gazebo composes them on top of mid_plate (z=0.07),
so the board, driver and top plate rendered floating at z~0.16-0.20 -
above the lidar. Fixed by using mid-plate-relative origins:

  gemstone/driver: 0.0225, top_plate: 0.06 -> absolutes 0.0925 / 0.13

Also the URDF->SDF conversion drops robot-level <material name> refs, so
the model rendered all gray. Added explicit <gazebo reference><material>
overrides per link (red battery, green PCB, blue driver, black lidar).

Verified in sim: gemstone z=0.0925, motor driver z=0.0925, top plate
z=0.13, lidar z=0.155; materials render (Gazebo/Red, /DarkGreen, /Blue);
/scan still returns office geometry (no sub-0.5 m self-occlusion).

Co-authored-by: alitalhq <alitqlhq@gmail.com>

File: src/gemstone_sim/urdf/gemstone_ugv_gazebo.xacro (robot description, xacro)
@@ -66,4 +66,11 @@
   <xacro:property name="driver_z" value="${board_z}"/>
   <xacro:property name="driver_mass" value="0.05"/>
+  <!-- mid_plate cizelgesi: gemstone/motor surucu/ust kapi mid_plate'in COCUGU
+       oldugu icin bu eklemlerin origin'leri mid_plate'e GORE (relative) olmali.
+       Dikkat: mutlak yukseklikler (board_z/top_plate_z) sadece base_link'in
+       dogrudan cocugu olan linklerde (lidar/camera/imu) kullanilabilir. -->
+  <xacro:property name="board_rel_z" value="${mid_plate_thickness/2 + board_thickness/2}"/>
+  <xacro:property name="driver_rel_z" value="${mid_plate_thickness/2 + driver_thickness/2}"/>
+  <xacro:property name="top_plate_rel_z" value="${top_plate_z - mid_plate_z}"/>
   <!-- Ust kapi tablasi (A1M8 lidar) -->
   <xacro:property name="top_plate_length" value="0.22"/>
@@ -246,5 +253,5 @@
     <parent link="mid_plate_link"/>
     <child link="gemstone_link"/>
-    <origin xyz="0 0 ${board_z}" rpy="0 0 0"/>
+    <origin xyz="0 0 ${board_rel_z}" rpy="0 0 0"/>
   </joint>
   <!-- Motor surucu: gemstone kartinin yaninda -->
@@ -269,5 +276,5 @@
     <parent link="mid_plate_link"/>
     <child link="motor_driver_link"/>
-    <origin xyz="${driver_x} 0 ${driver_z}" rpy="0 0 0"/>
+    <origin xyz="${driver_x} 0 ${driver_rel_z}" rpy="0 0 0"/>
   </joint>
   <!-- ===================== UST KAT: platform tablasi ===================== -->
@@ -292,5 +299,5 @@
     <parent link="mid_plate_link"/>
     <child link="top_plate_link"/>
-    <origin xyz="0 0 ${top_plate_z}" rpy="0 0 0"/>
+    <origin xyz="0 0 ${top_plate_rel_z}" rpy="0 0 0"/>
   </joint>
   <!-- A1M8 lidar: ust katin uzerinde, en tepede -->
@@ -487,8 +494,37 @@
     </plugin>
   </gazebo>
-  <!-- Gölgelendirme iyileştirmesi (isteğe bağlı görsel) -->
+  <!-- Görsel malzemeler. NOT: URDF <visual><material name="..."> referanslari
+       URDF->SDF donusumunde atilir (model gri render olur); bu yuzden her linke
+       acikca <gazebo reference><material> override'i verilir. -->
   <gazebo reference="base_link">
     <material>Gazebo/Gray</material>
   </gazebo>
+  <gazebo reference="mid_plate_link">
+    <material>Gazebo/Gray</material>
+  </gazebo>
+  <gazebo reference="top_plate_link">
+    <material>Gazebo/Gray</material>
+  </gazebo>
+  <gazebo reference="battery_link">
+    <material>Gazebo/Red</material>
+  </gazebo>
+  <gazebo reference="gemstone_link">
+    <material>Gazebo/DarkGreen</material>
+  </gazebo>
+  <gazebo reference="motor_driver_link">
+    <material>Gazebo/Blue</material>
+  </gazebo>
+  <gazebo reference="lidar_link">
+    <material>Gazebo/Black</material>
+  </gazebo>
+  <gazebo reference="camera_link">
+    <material>Gazebo/Black</material>
+  </gazebo>
+  <gazebo reference="imu_link">
+    <material>Gazebo/White</material>
+  </gazebo>
+  <gazebo reference="caster_wheel_link">
+    <material>Gazebo/White</material>
+  </gazebo>
   <gazebo reference="left_wheel_link">
     <material>Gazebo/DarkGrey</material>

Commit message: feat: caster wheel fix, Gazebo real-time factor, SLAM tuning for 5x, obstacle avoidance narrow corridor fix
- URDF: caster_wheel_joint fixed->continuous with friction, added to joint_state_publisher
- sim_bringup: add real_time_factor launch arg with Gazebo set_parameters service call
- auto_mapping: pass real_time_factor through to sim_bringup
- gcs.sh: set real_time_factor:=5.0 for simulation mode
- obstacle_avoidance: reduce safety_distance 0.30->0.25m and forward_half_angle 30->20 deg for narrow corridors
- SLAM toolbox: tune parameters for higher speed (scan_buffer 10->20, tf_buffer 30->60s, etc.)

File: src/gemstone_sim/urdf/gemstone_ugv_gazebo.xacro (robot description, xacro)
@@ -198,4 +198,12 @@
         <sphere radius="${caster_radius}"/>
       </geometry>
+      <surface>
+        <friction>
+          <ode>
+            <mu>1.0</mu>
+            <mu2>1.0</mu2>
+          </ode>
+        </friction>
+      </surface>
     </collision>
     <inertial>
@@ -204,8 +212,9 @@
     </inertial>
   </link>
-  <joint name="caster_wheel_joint" type="fixed">
+  <joint name="caster_wheel_joint" type="continuous">
     <parent link="base_link"/>
     <child link="caster_wheel_link"/>
     <origin xyz="${caster_x_offset} 0 ${caster_z_offset}" rpy="0 0 0"/>
+    <axis xyz="1 0 0"/>
   </joint>
   <!-- ===================== ORTA KAT: platform tablasi ===================== -->
@@ -492,4 +501,5 @@
       <joint_name>left_wheel_joint</joint_name>
       <joint_name>right_wheel_joint</joint_name>
+      <joint_name>caster_wheel_joint</joint_name>
     </plugin>
   </gazebo>
